Commit message: Moved wall closer. Added star png and made the image smaller.

File: urdf/ur10_cam.urdf.xacro (robot description, xacro)
@@ -319,6 +319,6 @@
     <joint name="camera_joint" type="fixed">
       <axis xyz="0 1 0" />
-      <origin xyz="0 0 ${shoulder_height}" rpy="0 0 0"/>
-      <parent link="${prefix}shoulder_link"/>
+      <origin xyz="0 0 ${shoulder_height}" rpy="0 -${pi / 2.0} 0"/>
+      <parent link="${prefix}wrist_1_link"/>
       <child link="camera_link"/>
     </joint>

Commit message: Fixed urdf, added motion control

File: urdf/ur10_cam.urdf.xacro (robot description, xacro)
@@ -85,5 +85,5 @@
       <parent link="${prefix}base_link" />
       <child link = "${prefix}shoulder_link" />
-      <origin xyz="0.0 0.0 ${shoulder_height}" rpy="0.0 0.0 -${pi / 2.0}" />
+      <origin xyz="0.0 0.0 ${shoulder_height}" rpy="0.0 0.0 0.0" />
       <axis xyz="0 0 1" />
       <xacro:unless value="${joint_limited}">
@@ -122,5 +122,5 @@
       <parent link="${prefix}shoulder_link" />
       <child link = "${prefix}upper_arm_link" />
-      <origin xyz="0.0 ${shoulder_offset} 0.0" rpy="0.0 0.0 0.0" />
+      <origin xyz="0.0 ${shoulder_offset} 0.0" rpy="0.0 ${pi / 2.0} 0.0" />
       <axis xyz="0 1 0" />
       <xacro:unless value="${joint_limited}">
@@ -159,5 +159,5 @@
       <parent link="${prefix}upper_arm_link" />
       <child link = "${prefix}forearm_link" />
-      <origin xyz="0.0 ${elbow_offset} ${upper_arm_length}" rpy="0.0 ${pi / 2.0} 0.0" />
+      <origin xyz="0.0 ${elbow_offset} ${upper_arm_length}" rpy="0.0 0.0 0.0" />
       <axis xyz="0 1 0" />
       <xacro:unless value="${joint_limited}">
@@ -196,5 +196,5 @@
       <parent link="${prefix}forearm_link" />
       <child link = "${prefix}wrist_1_link" />
-      <origin xyz="0.0 0.0 ${forearm_length}" rpy="0.0 0.0 0.0" />
+      <origin xyz="0.0 0.0 ${forearm_length}" rpy="0.0 ${pi / 2.0} 0.0" />
       <axis xyz="0 1 0" />
       <xacro:unless value="${joint_limited}">
@@ -318,6 +318,6 @@
     </link>
     <joint name="camera_joint" type="fixed">
-      <axis xyz="0 1 0" />
-      <origin xyz="0 0 ${shoulder_height}" rpy="0 -${pi / 2.0} 0"/>
+      <axis xyz="0 0 0" />
+      <origin xyz="0 0 ${shoulder_height}" rpy="0 -${pi} 0"/>
       <parent link="${prefix}wrist_1_link"/>
       <child link="camera_link"/>
